Commit message: Enhance UGV navigation and camera tracking functionalities
- Updated README to clarify waypoint selection behavior for file-based routes.
- Modified `run_follow_defaults.yaml` to adjust depth parameters and goal timing settings for improved performance.
- Refactored `sim_dataset_capture.py` to align camera pose topic naming conventions.
- Enhanced `camera_tracker.py` to publish additional camera target metrics and improve topic structure.
- Adjusted `follow_uav.py` and `follow_uav_odom.py` to streamline distance calculations and improve leader following logic.
- Implemented waypoint reordering in `ugv_nav2_driver.py` to ensure forward movement at the start of navigation.
- Added depth estimation improvements in `leader_estimator.py` with new rejection criteria for depth data.
- Updated `simulator.py` to refine camera pose publishing logic.
- Enhanced Xacro files for camera gimbal to support yaw and pitch joints with improved dynamics.

File: src/lrs_halmstad/xacro/lrs_camera_gimbal.sdf.xacro (robot description, xacro)
@@ -3,9 +3,9 @@
     <xacro:property name="M_PI" value="3.1415926535897931"/>
     <xacro:macro name="lrs_camera_gimbal"
-                 params="name parent_link link_name topic_base frame_id update_rate im_width im_height im_format hfov_deg far_clip robot_type robot_name x_offset:=0.0 y_offset:=0.0 z_offset:=0.0 pitch_offset:=0.0 yaw_offset:=0.0 sensor_roll_offset:=0.0 sensor_pitch_offset:=0.0 sensor_yaw_offset:=0.0">
+                 params="name parent_link link_name topic_base frame_id update_rate im_width im_height im_format hfov_deg far_clip robot_type robot_name x_offset:=0.0 y_offset:=0.0 z_offset:=0.0 pitch_offset:=0.0 yaw_offset:=0.0 sensor_roll_offset:=0.0 sensor_pitch_offset:=0.0 sensor_yaw_offset:=0.0 kinematic:=true">
       <link name="${link_name}">
          <pose rotation_format="euler_rpy" degrees="true">${x_offset} ${y_offset} ${z_offset} 0 ${pitch_offset} ${yaw_offset}</pose>
             <gravity>false</gravity>
-            <kinematic>true</kinematic>
+            <kinematic>${kinematic}</kinematic>
             <inertial>
                 <mass>0.01</mass>

File: src/lrs_halmstad/xacro/lrs_model.xacro (robot description, xacro)
@@ -87,8 +87,24 @@
     <xacro:if value="$(arg with_camera)">
         <xacro:property name="camera_prefix" value="/${base_name}/$(arg camera_name)"/>
+        <xacro:property name="camera_yaw_link_name" value="$(arg camera_name)_yaw_link"/>
         <xacro:property name="camera_link_name" value="$(arg camera_name)_link"/>
+        <link name="${camera_yaw_link_name}">
+            <pose rotation_format="euler_rpy" degrees="true">0 0 0 0 0 0</pose>
+            <gravity>false</gravity>
+            <inertial>
+                <mass>0.01</mass>
+                <inertia>
+                    <ixx>1.0e-4</ixx>
+                    <ixy>0.0</ixy>
+                    <ixz>0.0</ixz>
+                    <iyy>1.0e-4</iyy>
+                    <iyz>0.0</iyz>
+                    <izz>1.0e-4</izz>
+                </inertia>
+            </inertial>
+        </link>
         <xacro:include filename="$(find lrs_halmstad)/xacro/lrs_camera_gimbal.sdf.xacro"/>
         <xacro:lrs_camera_gimbal name="$(arg camera_name)"
-                                 parent_link="$(arg base_link_frame)"
+                                 parent_link="${camera_yaw_link_name}"
                                  link_name="${camera_link_name}"
                                  hfov_deg="$(arg camera_hfov)"
@@ -106,10 +122,29 @@
                                  robot_type="$(arg robot_type)"
                                  robot_name="$(arg name)"
+                                 kinematic="false"
                                  im_format="R8G8B8"
 />
-        <joint type="revolute" name="$(arg name)_gimbal_joint">
+        <joint type="revolute" name="$(arg name)_gimbal_yaw_joint">
+          <pose>0 0 0 0 0 0</pose>
+          <child>${camera_yaw_link_name}</child>
+          <parent>$(arg base_link_frame)</parent>
+          <axis>
+            <xyz>0 0 1</xyz>
+            <limit>
+              <lower>-3.1416</lower>
+              <upper>3.1416</upper>
+              <effort>100</effort>
+              <velocity>-1</velocity>
+            </limit>
+            <dynamics>
+              <damping>0.1</damping>
+            </dynamics>
+            <use_parent_model_frame>1</use_parent_model_frame>
+          </axis>
+        </joint>
+        <joint type="revolute" name="$(arg name)_gimbal_pitch_joint">
           <pose>0 0 0 0 0 0</pose>
           <child>${camera_link_name}</child>
-          <parent>$(arg base_link_frame)</parent>
+          <parent>${camera_yaw_link_name}</parent>
           <axis>
             <xyz>0 -1 0</xyz>
@@ -127,10 +162,18 @@
         </joint>
     <plugin
-      filename="ignition-gazebo-joint-position-controller-system"
-      name="ignition::gazebo::systems::JointPositionController">
+      filename="gz-sim-joint-position-controller-system"
+      name="gz::sim::systems::JointPositionController">
       <use_velocity_commands>true</use_velocity_commands>
       <joint_index>0</joint_index>
-      <joint_name>$(arg name)_gimbal_joint</joint_name>
+      <joint_name>$(arg name)_gimbal_pitch_joint</joint_name>
       <topic>/model/$(arg name)/joint/$(arg name)_gimbal_joint/pitch/cmd_pos</topic>
+    </plugin>
+    <plugin
+      filename="gz-sim-joint-position-controller-system"
+      name="gz::sim::systems::JointPositionController">
+      <use_velocity_commands>true</use_velocity_commands>
+      <joint_index>0</joint_index>
+      <joint_name>$(arg name)_gimbal_yaw_joint</joint_name>
+      <topic>/model/$(arg name)/joint/$(arg name)_gimbal_joint/yaw/cmd_pos</topic>
     </plugin>
     </xacro:if>
