Commit message: Add metadata and topics for YOLO experiment in warehouse
- Created metadata.json to store experiment details including start time, world, mode, UAV name, and topics.
- Added topics.txt listing all relevant ROS topics for the YOLO experiment.
- Introduced run_reset_experiment.sh script to reset the YOLO follow experiment without restarting Gazebo or Nav2, allowing for UAV and UGV teleportation and follow stack restart.

File: src/lrs_halmstad/clearpath/robot.urdf.xacro (robot description, xacro)
@@ -27,4 +27,9 @@
     <origin xyz="0.21 0.13 0.225" rpy="0.0 0.0 0.0"/>
   </xacro:hokuyo_ust>
+  <!-- camera_0 -->
+  <xacro:include filename="$(find clearpath_sensors_description)/urdf/intel_realsense.urdf.xacro"/>
+  <xacro:intel_realsense name="camera_0" parent_link="base_link" update_rate="30" image_height="480" image_width="640" model="d435">
+    <origin xyz="0.31 0.0 0.23" rpy="0.0 0.0 0.0"/>
+  </xacro:intel_realsense>
   <!-- Manipulators -->
   <!-- Extras -->
